File: Futbolista Castillo/HARDWARE/futbolista/futbolista.kicad_sch (KiCad schematic)
At the start: 12 parts, among them J1 Screw_Terminal_01x02, J2 Screw_Terminal_01x02, J3 Screw_Terminal_01x02, SW1 SW_DPST_x2, U1 HC-06, U2 L293D, U3 LM7805_TO220

Commit message: Add files via upload
Parts:
- added BZ1: Buzzer, EESTN5:Buzzer_12mm, symbol Device:Buzzer
- added D1, D2: LED, LED_THT:LED_D3.0mm, symbol Device:LED
- added Q1: 2N2222, 2N2222:TO127P584H533-3, symbol 2N2222:2N2222
- added R3: 330, Resistor_THT:R_Axial_DIN0204_L3.6mm_D1.6mm_P5.08mm_Horizontal, symbol Device:R
- added R4, R5: ~, Resistor_THT:R_Axial_DIN0204_L3.6mm_D1.6mm_P5.08mm_Horizontal, symbol Device:R
Connections:
- net +5V: now also A1.11 (D8), A1.12 (D9), R4.1, R5.1
- net 5volts arduino: now also BZ1.1 (+)
- net GND: now also D1.1 (K), D2.1 (K), Q1.1
- net D7: now reaches A1.5 (D2)
- net D7: now also R3.1
- new net: BZ1.2 (-), Q1.3
- new net: Q1.2, R3.2
- new net: D2.2 (A), R5.2
- new net: D1.2 (A), R4.2
Other:
- moved on the sheet: A1, SW1A, U3
