File: Futbolista Castillo/HARDWARE/futbolista/futbolista.kicad_pcb (KiCad board)
At the start: 2 copper layers, 12 parts, among them J1 Screw_Terminal_01x02, J2 Screw_Terminal_01x02, J3 Screw_Terminal_01x02, SW1 SW_DPST_x2, U1 HC-06, U2 L293D, U3 LM7805_TO220

Commit message: Add files via upload
Parts:
- added BZ1: Buzzer, EESTN5:Buzzer_12mm, F.Cu at (115.9, 99.1)
- added D1: LED, LED_THT:LED_D3.0mm, F.Cu at (111.0, 80.6)
- added D2: LED, LED_THT:LED_D3.0mm, F.Cu at (111.0, 87.0)
- added Q1: 2N2222, 2N2222:TO127P584H533-3, F.Cu at (118.4, 109.6)
- added R3: 330, Resistor_THT:R_Axial_DIN0204_L3.6mm_D1.6mm_P5.08mm_Horizontal, F.Cu at (121.5, 116.0)
- added R4: ~, Resistor_THT:R_Axial_DIN0204_L3.6mm_D1.6mm_P5.08mm_Horizontal, F.Cu at (123.1, 80.7)
- added R5: ~, Resistor_THT:R_Axial_DIN0204_L3.6mm_D1.6mm_P5.08mm_Horizontal, F.Cu at (123.1, 87.0)
- moved R2 81.3 mm to (99.1, 109.2), turned to 0 degrees
- moved R1 74.3 mm to (104.1, 112.2), turned to 180 degrees
- moved U1 65.5 mm to (108.1, 107.3), turned to 90 degrees
- moved U3 36.0 mm to (173.8, 102.4), turned to 0 degrees
- moved J2 33.0 mm to (154.7, 113.3)
- moved C2 32.9 mm to (155.0, 104.1)
- moved U2 32.7 mm to (148.6, 100.3)
- moved C1 32.7 mm to (160.0, 89.1)
- moved J1 32.6 mm to (160.2, 80.9)
- moved SW1 31.8 mm to (177.2, 91.1), turned to -90 degrees
- moved J3 29.1 mm to (191.1, 102.3), turned to 90 degrees
- moved A1 28.3 mm to (142.2, 119.4)
Connections:
- A1 pad 11: unconnected-(A1-D8-Pad11) -> D8
- A1 pad 12: unconnected-(A1-D9-Pad12) -> D8
- A1 pad 5: unconnected-(A1-D2-Pad5) -> D7
- U1 pad P$5: +5V -> D8
- U2 pad 16: +5V -> D8
- U3 pad 3: +5V -> D8
Routing:
- net +5V: track 110.5 -> 0.00 mm
- net ENABLE2: track 70.9 -> 28.5 mm
- net D8: track 0.00 -> 39.3 mm
- net D7: track 0.00 -> 36.9 mm
- net GND: track 31.1 -> 0.00 mm, vias 2 -> 0
- net VCC: track 43.5 -> 22.9 mm
- net 5volts arduino: track 0.00 -> 19.4 mm
- net Net-(BZ1--): track 0.00 -> 15.2 mm
- net Net-(Q1-Pad2): track 0.00 -> 8.44 mm
- net B3: track 44.8 -> 37.0 mm
- net A2: track 45.6 -> 39.8 mm
- net ENABLE1: track 11.6 -> 6.89 mm
- net Net-(D1-A): track 0.00 -> 4.53 mm
- net Net-(D2-A): track 0.00 -> 4.48 mm
- net Net-(J3-Pin_2): track 10.5 -> 14.6 mm
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
Commit message: Add files via upload
Routing:
- net D8: track 39.3 -> 190.5 mm
- net GND: track 0.00 -> 4.50 mm, vias 0 -> 2
Changed lines of the file:
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@@
+	)
+	(segment
+		(start 106 114.5)
+		(end 106 110)
+		(width 1.5)
+		(layer "F.Cu")
+		(net 10)
+	)
+	(via
+		(at 106 110)
+		(size 0.6)
+		(drill 0.3)
+		(layers "F.Cu" "B.Cu")
+		(free yes)
+		(net 10)
+	)
+	(via
+		(at 106 114.5)
+		(size 0.6)
+		(drill 0.3)
+		(layers "F.Cu" "B.Cu")
+		(free yes)
+		(net 10)
+	)
+	(segment
+		(start 102.489 108.542883)
+		(end 102.489 109.910617)
+		(width 1.5)
+		(layer "B.Cu")
+		(net 13)
+	)
+	(segment
+		(start 92.09725 111.59725)
+		(end 92.09725 89.90275)
+		(width 1.5)
+		(layer "B.Cu")
+		(net 13)
+	)
+	(segment
+		(start 93.159 88.841)
+		(end 122.659 88.841)
+		(width 1.5)
+		(layer "B.Cu")
+		(net 13)
 	)
 	(segment
@@
 	)
 	(segment
+		(start 179.8965 78.8965)
+		(end 179.8965 101.3535)
+		(width 0.75)
+		(layer "B.Cu")
+		(net 13)
+	)
+	(segment
 		(start 142.24 91.44)
 		(end 142.24 93.98)
@@
 	)
 	(segment
-		(start 144.8 91.44)
-		(end 142.24 91.44)
-		(width 0.75)
+		(start 94.36775 113.86775)
+		(end 92.09725 111.59725)
+		(width 1.5)
+		(layer "B.Cu")
+		(net 13)
+	)
+	(segment
+		(start 102.489 111.532883)
+		(end 102.489 112.511)
+		(width 1.5)
+		(layer "B.Cu")
+		(net 13)
+	)
+	(segment
+		(start 103.90675 105.63675)
+		(end 103.90675 106.714867)
+		(width 1.5)
 		(layer "B.Cu")
 		(net 13)
@@
 	)
 	(segment
-		(start 146.065 92.705)
-		(end 144.8 91.44)
+		(start 102.5 111.521883)
+		(end 102.489 111.532883)
+		(width 1.5)
+		(layer "B.Cu")
+		(net 13)
+	)
+	(segment
+		(start 122.659 88.841)
+		(end 123.11 88.39)
+		(width 1.5)
+		(layer "B.Cu")
+		(net 13)
+	)
+	(segment
+		(start 123.11 88.39)
+		(end 123.11 86.99)
+		(width 1.5)
+		(layer "B.Cu")
+		(net 13)
+	)
+	(segment
+		(start 179.8965 101.3535)
+		(end 178.87 102.38)
+		(width 0.75)
+		(layer "B.Cu")
+		(net 13)
+	)
+	(segment
+		(start 140.864 89.469958)
+		(end 140.864 78.636)
 		(width 0.75)
 		(layer "B.Cu")
@@
 	(segment
 		(start 148.59 92.705)
-		(end 146.065 92.705)
-		(width 0.75)
+		(end 144.099042 92.705)
+		(width 0.75)
+		(layer "B.Cu")
+		(net 13)
+	)
+	(segment
+		(start 101.13225 113.86775)
+		(end 94.36775 113.86775)
+		(width 1.5)
 		(layer "B.Cu")
 		(net 13)
@@
 	)
 	(segment
+		(start 140.864 78.636)
+		(end 142.077 77.423)
+		(width 0.75)
+		(layer "B.Cu")
+		(net 13)
+	)
+	(segment
+		(start 102.5 108.121617)
+		(end 102.5 108.531883)
+		(width 1.5)
+		(layer "B.Cu")
+		(net 13)
+	)
+	(segment
+		(start 102.489 112.511)
+		(end 101.13225 113.86775)
+		(width 1.5)
+		(layer "B.Cu")
+		(net 13)
+	)
+	(segment
+		(start 103.90675 106.714867)
+		(end 102.5 108.121617)
+		(width 1.5)
+		(layer "B.Cu")
+		(net 13)
+	)
+	(segment
+		(start 178.423 77.423)
+		(end 179.8965 78.8965)
+		(width 0.75)
+		(layer "B.Cu")
+		(net 13)
+	)
+	(segment
 		(start 123.11 86.99)
 		(end 123.11 80.67)
@@
 		(layer "B.Cu")
 		(net 13)
+	)
+	(segment
+		(start 102.5 108.531883)
+		(end 102.489 108.542883)
+		(width 1.5)
+		(layer "B.Cu")
+		(net 13)
+	)
+	(segment
+		(start 102.489 109.910617)
+		(end 102.5 109.921617)
+		(width 1.5)
+		(layer "B.Cu")
+		(net 13)
+	)
+	(segment
+		(start 142.077 77.423)
+		(end 178.423 77.423)
+		(width 0.75)
+		(layer "B.Cu")
+		(net 13)
+	)
+	(segment
+		(start 102.5 109.921617)
+		(end 102.5 111.521883)
+		(width 1.5)
+		(layer "B.Cu")
+		(net 13)
+	)
+	(segment
+		(start 144.099042 92.705)
+		(end 140.864 89.469958)
+		(width 0.75)
+		(layer "B.Cu")
+		(net 13)
+	)
+	(segment
+		(start 92.09725 89.90275)
+		(end 93.159 88.841)
+		(width 1.5)
+		(layer "B.Cu")
+		(net 13)
